File: pcb/with-regulators/cvbs-camera-module-with-regulators.kicad_sch (KiCad schematic)
At the start: 17 parts, among them J1 X.FL-PR-SMT1-2(80), J2 5052740612, J3 U.FL-R-SMT(10), J5 Conn_01x03, J6 U.FL-R-SMT(10), U1 cvbs-camera, U2 TPS8269xxxSIPR, U3 NCP163AFCT250T2G

Commit message: Address feedback
- Fill out title blocks
- LEDs 0201 -> 0402 & assign PN
- Power LEDs with 2.85V regulator
- Remove noise on fab layers
- Thicken flex cable
- Add .sldprt & .dxf files for flex pattern
Parts:
- D1, D2, D3: value LED -> IN-S42CTQIR; footprint LED_SMD:LED_0201_0603Metric -> LED_SMD:LED_0402_1005Metric
- J3, J6: value U.FL-R-SMT(10) -> X.FL-R-SMT-1(02); footprint Connector_Coaxial:U.FL_Hirose_U.FL-R-SMT-1_Vertical -> jonnew:HIROSE_X.FL-R-SMT-1
- U2: value TPS8269xxxSIPR -> TPS82693SIPR; symbol open-ephys:TPS8269xxxSIPR -> open-ephys:TPS8269x
Connections:
- net +2V5: no longer J5.1 (Pin_1), R1.1, R2.1, R3.1
- net VCC: now also J5.1 (Pin_1)
- net +2V8: now reaches C1.1, U2.A1 (VOUT), U3.A1 (VIN), U3.B1 (EN)
- net +2V8: now also R1.1, R2.1, R3.1
