File: pcb/without-regulators/cvbs-camera-module.kicad_sch (KiCad schematic)
At the start: 13 parts, among them J1 X.FL-PR-SMT1-2(80), J2 5052740612, J3 X.FL-R-SMT-1(02), J5 Conn_01x03, J6 X.FL-R-SMT-1(02), U1 cvbs-camera

Commit message: Address feedback
- Fill out title blocks
- LEDs 0201 -> 0402 & assign PN
- Power LEDs with 2.85V regulator
- Remove noise on fab layers
- Thicken flex cable
- Add .sldprt & .dxf files for flex pattern
Parts:
- D1, D2, D3: value LED -> IN-S42CTQIR; footprint LED_SMD:LED_0201_0603Metric -> LED_SMD:LED_0402_1005Metric
Other:
- company: (none) -> Open Ephys
- title: (none) -> NP2E-CVBS-EXTENSION
Changed lines of the file:
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@@
 	(generator_version "10.0")
 	(paper "A3")
+	(title_block
+		(title "NP2E-CVBS-EXTENSION")
+		(date "2026-06-09")
+		(rev "A")
+		(company "Open Ephys")
+	)
 	(rectangle
 		(start 114.3 177.8)
@@
 			)
 		)
-		(property "Value" "LED"
+		(property "Value" "IN-S42CTQIR"
 			(at 242.8875 223.52 0)
 			(show_name no)
@@
 			)
 		)
-		(property "Footprint" "LED_SMD:LED_0201_0603Metric"
+		(property "Footprint" "LED_SMD:LED_0402_1005Metric"
 			(at 241.3 228.6 0)
 			(hide yes)
@@
 			)
 		)
-		(property "Value" "LED"
+		(property "Value" "IN-S42CTQIR"
 			(at 242.8875 236.22 0)
 			(show_name no)
@@
 			)
 		)
-		(property "Footprint" "LED_SMD:LED_0201_0603Metric"
+		(property "Footprint" "LED_SMD:LED_0402_1005Metric"
 			(at 241.3 241.3 0)
 			(hide yes)
@@
 			)
 		)
-		(property "Value" "LED"
+		(property "Value" "IN-S42CTQIR"
 			(at 242.8875 210.82 0)
 			(show_name no)
@@
 			)
 		)
-		(property "Footprint" "LED_SMD:LED_0201_0603Metric"
+		(property "Footprint" "LED_SMD:LED_0402_1005Metric"
 			(at 241.3 215.9 0)
 			(hide yes)
